File: kicad/kicad.kicad_pcb (KiCad board)
At the start: 2 copper layers, 11 parts, among them U1 ProMicro

Commit message: cccc
Parts:
- added S1: MX_stab, marbastlib-mx:STAB_MX_2.25u, F.Cu at (95.0, 106.5)
- moved U1 155.4 mm to (38.1, 61.4), turned to -90 degrees
- moved MX7 70.0 mm to (82.2, 87.6)
- moved MX9 36.4 mm to (57.9, 106.5)
- moved MX10 18.4 mm to (95.2, 106.6)
- moved MX8 15.4 mm to (106.4, 87.5)
- moved MX6 0.77 mm to (57.9, 87.5)
