File: kicad/kicad.kicad_sch (KiCad schematic)
At the start: 0 parts

Commit message: hehe new uppp
Parts:
- added MX1, MX10, MX2, MX3, MX4, MX5, MX6, MX7, MX8, MX9: MX_SW_HS, MX_Only:MXOnly-1.25U-Hotswap-LED, symbol marbastlib-mx:MX_SW_HS_KS-2P02B01-01
- added S1: MX_stab, PCM_marbastlib-mx:STAB_MX_P_6.25u, symbol marbastlib-mx:MX_stab
- added U1: ProMicro, Keebio-Parts:ArduinoProMicro, symbol keebio:ProMicro

Commit message: cccc
Parts:
- S1: footprint PCM_marbastlib-mx:STAB_MX_P_6.25u -> marbastlib-mx:STAB_MX_2.25u
Connections:
- net GND: now reaches U1.23 (GND)
- net GND: now also MX1.2, MX10.2, MX3.2, MX4.2, MX5.2, MX6.2, MX7.2, MX8.2, MX9.2, U1.3 (GND), U1.4 (GND)
Other:
- moved on the sheet: MX1, MX10, MX3, MX4, MX5, MX7
